File: aistompboxadapter.kicad_sch (KiCad schematic)
At the start: 25 parts, among them J1 SYNTH IN, J2 FX RETURN, J3 Synth Power, J4 FX SEND, J5 SYNTH OUT, U1 TL072

Commit message: smd and add fab files
Parts:
- removed C4, C5: 100n, Sonosus:C_Disc_D3.0mm_W2.0mm_P2.50mm, symbol Device:C_Small
- removed H2: MountingHole, MountingHole:MountingHole_3.2mm_M3, symbol Mechanical:MountingHole
- C2: footprint Sonosus:C_Rect_L7.0mm_W2.5mm_P5.00mm -> Capacitor_SMD:C_0805_2012Metric; LCSC (none) -> C1785
- C6: footprint Sonosus:C_Rect_L7.0mm_W2.5mm_P5.00mm -> Capacitor_SMD:C_0805_2012Metric; LCSC (none) -> C14857
- D1, D2: footprint Diode_THT:D_DO-41_SOD81_P10.16mm_Horizontal -> Diode_THT:D_DO-41_SOD81_P2.54mm_Vertical_KathodeUp
- J1: value SYNTH IN -> SI
- R1: footprint Sonosus:R_Axial_DIN0207_L6.3mm_D2.5mm_P7.62mm_Horizontal -> Resistor_SMD:R_0805_2012Metric; LCSC (none) -> C17514
- R2: footprint Sonosus:R_Axial_DIN0207_L6.3mm_D2.5mm_P7.62mm_Horizontal -> Resistor_SMD:R_0805_2012Metric; LCSC (none) -> C17470
- R3: footprint Sonosus:R_Axial_DIN0207_L6.3mm_D2.5mm_P7.62mm_Horizontal -> Resistor_SMD:R_0805_2012Metric; LCSC (none) -> C17560
- R4, R7: footprint Sonosus:R_Axial_DIN0207_L6.3mm_D2.5mm_P7.62mm_Horizontal -> Resistor_SMD:R_0805_2012Metric; LCSC (none) -> C17513
- R5: footprint Sonosus:R_Axial_DIN0207_L6.3mm_D2.5mm_P7.62mm_Horizontal -> Resistor_SMD:R_0805_2012Metric; LCSC (none) -> C17710
- R6: footprint Sonosus:R_Axial_DIN0207_L6.3mm_D2.5mm_P7.62mm_Horizontal -> Resistor_SMD:R_0805_2012Metric; LCSC (none) -> C17414
- U1: footprint Sonosus:DIP-8_W7.62mm_Socket_LongPads -> Package_SO:SOIC-8_3.9x4.9mm_P1.27mm; LCSC (none) -> C6961
